Commit message: fixing errors

File: polaris_gem_simulator/gem_simulator/gem_description/urdf/gem.urdf.xacro (robot description, xacro)
@@ -65,10 +65,12 @@
   </link>
   <!-- ***************************************** Set vehicle load point ***************************************** -->
-  <joint name="base_link" type="fixed">
+  <!-- joint name="base_link" type="fixed" -->
+  <joint name="base_footprint_to_base_link" type="fixed">
     <origin xyz="0 0 0.44" rpy="0 0 0"/>
     <parent link="base_footprint"/>
     <child link="base_link"/>
   </joint>
-  <joint name="center_link" type="fixed">
+  <!-- joint name="center_link" type="fixed" -->
+  <joint name="base_link_to_center_link" type="fixed">
     <origin xyz="0.87 0 0.151" rpy="0 0 0"/>
     <parent link="base_link"/>
